File: spacey.kicad_sch (KiCad schematic)
At the start: 1 part, among them P1 USB_C_Plug_USB2.0

Commit message: Finished PCB
Parts:
- removed P1: USB_C_Plug_USB2.0, symbol Connector:USB_C_Plug_USB2.0
- added D1, D2, D3, D4: WS2813, LED_SMD:LED_WS2812_PLCC6_5.0x5.0mm_P1.6mm, symbol LED:WS2813
- added J1: Screw_Terminal_01x02, TerminalBlock_4Ucon:TerminalBlock_4Ucon_1x02_P3.50mm_Horizontal, symbol Connector:Screw_Terminal_01x02
- added SW1, SW10, SW2, SW3, SW4, SW5, SW6, SW7, SW8, SW9: SW_Omron_B3FS, Button_Switch_THT:SW_TH_Tactile_Omron_B3F-10xx, symbol Switch:SW_Omron_B3FS
- added U1: XIAO-nRF52840-SMD, Seeed Studio XIAO Series Library:XIAO-nRF52840-SMD, symbol Seeed_Studio_XIAO_Series:XIAO-nRF52840-SMD
Connections:
- new net: D3.3 (DOUT), D4.4 (DIN)
- new net: D2.3 (DOUT), D3.4 (DIN)
- new net: D1.3 (DOUT), D2.4 (DIN)
- new net +3V3: U1.12 (3V3)
- new net +5V: D1.2 (VDD), D2.2 (VDD), D3.2 (VDD), D4.2 (VDD), U1.14 (5V)
- new net +BATT: J1.1 (Pin_1), U1.15 (BAT)
- new net DIN: D1.4 (DIN), U1.6 (P0.05_A5_D5_SCL)
- new net GND: D1.5 (GND), D2.5 (GND), D3.5 (GND), D4.5 (GND), J1.2 (Pin_2), SW1.1, SW10.1, SW2.1, SW3.1, SW4.1, SW5.1, SW6.1, SW7.1, SW8.1, SW9.1, U1.13 (GND), U1.16 (GND), U1.22 (GND)
- new net bt_1: SW2.2, U1.7 (P1.11_D6_TX)
- new net bt_10: SW10.2, U1.11 (P1.15_D10_MOSI)
- new net bt_2: SW4.2, U1.5 (P0.04_A4_D4_SDA)
- new net bt_3: SW6.2, U1.4 (P0.29_A3_D3)
- new net bt_4: SW5.2, U1.3 (P0.28_A2_D2)
- new net bt_5: SW3.2, U1.2 (P0.03_A1_D1)
- new net bt_6: SW1.2, U1.1 (P0.02_A0_D0)
- new net bt_7: SW9.2, U1.8 (P1.12_D7_RX)
- new net bt_8: SW7.2, U1.9 (P1.13_D8_SCK)
- new net bt_9: SW8.2, U1.10 (P1.14_D9_MISO)
- no-connect marks 0 -> 11
